File: elrs_tx_full.kicad_sch (KiCad schematic)
At the start: 9 parts, among them J2 DEBUG, J3 RUN, J4 DC_DC, U1 E28-2G4M27S-MY, U2 ESP32-WROOM-32-MY

Commit message: pcb progress
Parts:
- added J1: LED Chain, Connector_PinHeader_2.54mm:PinHeader_1x01_P2.54mm_Vertical, symbol Connector_Generic:Conn_01x01
- added J5: OLED_I2C, Connector_PinHeader_2.54mm:PinHeader_1x04_P2.54mm_Vertical, symbol Connector_Generic:Conn_01x04
Connections:
- net +3.3V: now also D1.1 (VDD), J5.2 (Pin_2)
- net GND: now also D1.3 (VSS), J5.1 (Pin_1)
- net LED_RGB: now also D1.4 (DIN)
- net OLED_SDA: now reaches U2.8 (IO32)
- net OLED_SDA: now also J5.4 (Pin_4)
- net OLED_SCK: now reaches U2.9 (IO33)
- net OLED_SCK: now also J5.3 (Pin_3)
- net at D1.2 (DOUT): now also J1.1 (Pin_1)
Other:
- moved on the sheet: D1

Commit message: pcb progress
Parts:
- J4: footprint Connector_PinHeader_2.54mm:PinHeader_1x04_P2.54mm_Vertical -> elrs_tx_full:DC_DC_20x11
Changed lines of the file:
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@@
 			)
 		)
-		(property "Footprint" "Connector_PinHeader_2.54mm:PinHeader_1x04_P2.54mm_Vertical"
+		(property "Footprint" "elrs_tx_full:DC_DC_20x11"
 			(at 99.06 184.15 0)
 			(effects

Commit message: pcb progress
Parts:
- added C2, C3: 10uF, Capacitor_SMD:C_1206_3216Metric_Pad1.33x1.80mm_HandSolder, symbol Device:C
- added H1, H2, H3, H4: MountingHole, MountingHole:MountingHole_2.2mm_M2_Pad, symbol Mechanical:MountingHole
- added J10: IO3, Connector_PinHeader_1.27mm:PinHeader_1x03_P1.27mm_Vertical, symbol Connector_Generic:Conn_01x03
- added J6: RUN, Connector_PinHeader_2.54mm:PinHeader_1x03_P2.54mm_Vertical, symbol Connector_Generic:Conn_01x03
- added J7: IO1, Connector_PinHeader_1.27mm:PinHeader_1x02_P1.27mm_Vertical, symbol Connector_Generic:Conn_01x02
- added J8: DEBUG, Connector_PinHeader_2.54mm:PinHeader_1x05_P2.54mm_Vertical, symbol Connector_Generic:Conn_01x05
- added J9: IO2, Connector_PinHeader_1.27mm:PinHeader_1x02_P1.27mm_Vertical, symbol Connector_Generic:Conn_01x02
- added P1: USB_C_Plug_USB2.0, elrs_tx_full:USB_C_DEALON_009, symbol Connector:USB_C_Plug_USB2.0
- J2: footprint Connector_PinHeader_2.54mm:PinHeader_1x05_P2.54mm_Vertical -> Connector_JST:JST_PH_S5B-PH-SM4-TB_1x05-1MP_P2.00mm_Horizontal
- J3: footprint Connector_PinHeader_2.54mm:PinHeader_1x03_P2.54mm_Vertical -> Connector_JST:JST_PH_S3B-PH-SM4-TB_1x03-1MP_P2.00mm_Horizontal
- J5: footprint Connector_PinHeader_2.54mm:PinHeader_1x04_P2.54mm_Vertical -> elrs_tx_full:OLED_27.3x27.8mm_no_holes
- U2: footprint elrs_tx_full:ESP32-WROOM-32D-MY -> elrs_tx_full:ESP32-WROOM-32_zhaw
Connections:
- net +3.3V: now also C2.1, C3.1, J8.2 (Pin_2)
- net +BATT: now also J6.2 (Pin_2), P1.A4 (VBUS), P1.A9 (VBUS), P1.B4 (VBUS), P1.B9 (VBUS)
- net CRSF_RX_TX: now also J6.3 (Pin_3)
- net ESP32_BOOT0: now also J8.5 (Pin_5)
- net ESP32_RX: now also J8.4 (Pin_4)
- net ESP32_TX: now also J8.3 (Pin_3)
- net GND: now also C2.2, C3.2, J6.1 (Pin_1), J8.1 (Pin_1), P1.A1 (GND), P1.A12 (GND), P1.B1 (GND), P1.B12 (GND)
- net IO25: now reaches U2.10 (IO25)
- net IO25: now also J9.1 (Pin_1)
- net IO12: now reaches U2.14 (IO12)
- net IO12: now also J9.2 (Pin_2)
- net IO16: now reaches U2.27 (IO16)
- net IO16: now also J10.1 (Pin_1)
- net IO17: now reaches U2.28 (IO17)
- net IO17: now also J10.2 (Pin_2)
- net IO22: now reaches U2.36 (IO22)
- net IO22: now also J10.3 (Pin_3)
- net IO34: now reaches U2.6 (IO34)
- net IO34: now also J7.1 (Pin_1)
- net IO35: now reaches U2.7 (IO35)
- net IO35: now also J7.2 (Pin_2)
- no-connect marks 7 -> 14
Other:
- moved on the sheet: C1, D1, J1, J2, J3, J4, J5

Commit message: pcb progress
Parts:
- added C9: 10uF, Capacitor_SMD:C_1206_3216Metric_Pad1.33x1.80mm_HandSolder, symbol Device:C
- added R3: 56k, Resistor_SMD:R_0805_2012Metric_Pad1.20x1.40mm_HandSolder, symbol Device:R
- added R4: 22k, Resistor_SMD:R_0805_2012Metric_Pad1.20x1.40mm_HandSolder, symbol Device:R
- added SW1: RESET, Button_Switch_SMD:SW_SPST_EVQP0, symbol Switch:SW_Push
- added U3: SPX3819M5-L, Package_TO_SOT_SMD:SOT-23-5, symbol Regulator_Linear:SPX3819M5-L
Connections:
- net +3.3V: no longer D1.1 (VDD)
- net +BATT: now also U3.1 (IN), U3.3 (EN)
- net GND: now also C9.2, R4.2, SW1.1, U3.2 (GND)
- net EN: now reaches R2.1, U2.3 (EN)
- net EN: now also C9.1, SW1.2
- new net: R3.2, R4.1, U3.4 (ADJ)
- new net +5V: D1.1 (VDD), R3.1, U3.5 (OUT)
Other:
- note added: "Additional Pins"
- note added: "DC-DC 12V -> 3.3V 3A"
- note added: "Debug"
- note added: "Enable"
- note added: "LDO 12V -> 4.37 500 mA"
- note added: "Microcontroller ESP32"
- note added: "OLED Display"
- note added: "RGB-LED"
- note added: "Radio"
- note added: "Remote Control"
- note added: "USB-C"
- moved on the sheet: C1, C2, C3, D1, J1, J10, J2, J3, J4, J5, J6, J7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
